File: D8_schematic.brd (EAGLE design)
At the start: 53.1 x 68.8 mm, 14 parts

Commit message: Add files via upload
Routing:
- net N$13: track 79.9 -> 26.3 mm
- net N$3: track 67.5 -> 26.6 mm
- net N$5: track 32.1 -> 60.4 mm
- net N$10: track 71.1 -> 48.3 mm
- net N$12: track 47.1 -> 67.3 mm
- net N$6: track 53.5 -> 35.1 mm
- net N$2: track 44.6 -> 58.2 mm
- net N$4: track 33.6 -> 26.6 mm
- net N$9: track 19.6 -> 17.1 mm
- net N$1: track 29.6 -> 29.0 mm
